File: schematic/diode_logic_schematic.kicad_sch (KiCad schematic)
At the start: 14 parts, among them K1 i2c_LCD

Commit message: move schematic, add image
Other:
- note removed: "Select logic"
- company: (none) -> BYU
- title: (none) -> Photodiode-based Logic Puzzle
- moved on the sheet: A1, D1, D2, D3, D4, D5, D6, K1, R1, R2, R3, R4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
